Commit message: ..

File: urdf/arm.xacro (robot description, xacro)
@@ -33,19 +33,18 @@
     <!--     <xacro:property name="pi" value="3.141592654" /> -->
     <xacro:property name="M_PI" value="3.141592654"/>
-    <xacro:property name="l4" value="0.05"/>
-    <xacro:property name="width" value="0.05"/>
     <xacro:property name="joint_radius" value="0.05"/>
     <xacro:property name="joint_height" value="0.2"/>
+    <xacro:property name="width" value="0.05"/>
     <xacro:property name="l1" value="0.3"/>
-    <xacro:property name="l2" value="0.3"/>
-    <xacro:property name="l3" value="0.3"/>
+    <xacro:property name="l2" value="1"/>
+    <xacro:property name="l3" value="0.8"/>
     <xacro:property name="l4" value="0.2"/>
     <xacro:property name="l5" value="0.2"/>
-    <xacro:property name="l6" value="0.3"/>
-    <xacro:property name="end_ball_radius" value="0.05"/>
+    <xacro:property name="l6" value="0.2"/>
+    <xacro:property name="end_ball_radius" value="0.025"/>
     <!-- Used for fixing robot to Gazebo 'link 1' -->
     <link name="world"/>
     <joint name="j1" type="revolute">
-        <origin xyz="0 0 0" rpy="0 0 0"/>
+        <origin xyz="0 0 0.15" rpy="0 0 0"/>
         <parent link="world"/>
         <child link="joint1"/>
@@ -73,5 +72,5 @@
         </inertial>
     </link>
-<!--    <joint name="link1_fix" type="fixed">
+    <joint name="link1_fix" type="fixed">
         <origin xyz="0 0 0" rpy="0 0 0"/>
         <parent link="joint1"/>
@@ -98,7 +97,6 @@
         </inertial>
     </link>
-   -->
     <joint name="j2" type="revolute">
-        <origin xyz="0 0 ${l1}" rpy="${pi*0.5} ${pi*0.0} ${pi*0.5}"/>
+        <origin xyz="0 0 ${l1}" rpy="${pi*0.0} ${pi*0.5} ${pi*0.0}"/>
         <parent link="joint1"/>
         <child link="joint2"/>
@@ -126,5 +124,5 @@
         </inertial>
     </link>
-<!--    <joint name="link2_fix" type="fixed">
+    <joint name="link2_fix" type="fixed">
         <origin xyz="0 0 0" rpy="0 0 0"/>
         <parent link="joint2"/>
@@ -151,5 +149,4 @@
         </inertial>
     </link>
-    -->
     <joint name="j3" type="revolute">
         <origin xyz="0 ${l2} 0" rpy="${pi*0.0} ${pi*0.0} ${pi*0.5}"/>
@@ -179,5 +176,5 @@
         </inertial>
     </link>
-<!--    <joint name="link3_fix" type="fixed">
+    <joint name="link3_fix" type="fixed">
         <origin xyz="0 0 0" rpy="0 0 0"/>
         <parent link="joint3"/>
@@ -204,5 +201,4 @@
         </inertial>
     </link>
-    -->
     <joint name="j4" type="revolute">
         <origin xyz="${l3} 0 0" rpy="${pi*0.5} ${pi*0} ${pi*0.5}"/>
@@ -232,5 +228,5 @@
         </inertial>
     </link>
-<!--    <joint name="link4_fix" type="fixed">
+    <joint name="link4_fix" type="fixed">
         <origin xyz="0 0 0" rpy="0 0 0"/>
         <parent link="joint4"/>
@@ -257,5 +253,4 @@
         </inertial>
     </link>
-    -->
     <joint name="j5" type="revolute">
         <origin xyz="0 0 ${l4}" rpy="${-pi*0.5} ${pi*1} ${pi*0.0}"/>
@@ -285,5 +280,5 @@
         </inertial>
     </link>
-<!--    <joint name="link5_fix" type="fixed">
+    <joint name="link5_fix" type="fixed">
         <origin xyz="0 0 0" rpy="0 0 0"/>
         <parent link="joint5"/>
@@ -310,5 +305,4 @@
         </inertial>
     </link>
-    -->
     <joint name="j6" type="revolute">
         <origin xyz="0 ${l5} 0" rpy="${-pi*0.5} ${pi*1} ${pi*0.0}"/>
@@ -338,7 +332,6 @@
         </inertial>
     </link>
-    <!--
     <joint name="link6_fix" type="fixed">
-        <origin xyz="0 0 0" rpy="0 0 0"/>
+        <origin xyz="0 0 ${l6}" rpy="0 0 0"/>
         <parent link="joint6"/>
         <child link="link6"/>
@@ -346,5 +339,5 @@
     <link name="link6">
         <collision>
-            <origin xyz="0 0 ${l6}" rpy="0 0 0"/>
+            <origin xyz="0 0 0" rpy="0 0 0"/>
             <geometry>
                 <sphere radius="${end_ball_radius}" />
@@ -352,5 +345,5 @@
         </collision>
         <visual>
-            <origin xyz="0 0 ${l6}" rpy="0 0 0"/>
+            <origin xyz="0 0 0" rpy="0 0 0"/>
             <geometry>
                 <sphere radius="${end_ball_radius}" />
@@ -364,4 +357,84 @@
         </inertial>
     </link>
-    -->
+    <gazebo reference="link1">
+        <material>Gazebo/DarkGrey</material>
+    </gazebo>
+    <gazebo reference="link2">
+        <material>Gazebo/FlatBlack</material>
+    </gazebo>
+    <gazebo reference="link3">
+        <material>Gazebo/DarkGrey</material>
+    </gazebo>
+    <gazebo reference="link4">
+        <material>Gazebo/FlatBlack</material>
+    </gazebo>
+    <gazebo reference="link5">
+        <material>Gazebo/DarkGrey</material>
+    </gazebo>
+    <gazebo reference="link6">
+        <material>Gazebo/FlatBlack</material>
+    </gazebo>
+    <transmission name="transmission">
+        <type>transmission_interface/SimpleTransmission</type>
+        <joint name="j1">
+            <hardwareInterface>hardware_interface/EffortJointInterface</hardwareInterface>
+        </joint>
+        <actuator name="motor1">
+            <hardwareInterface>hardware_interface/EffortJointInterface</hardwareInterface>
+            <mechanicalReduction>1</mechanicalReduction>
+        </actuator>
+    </transmission>
+    <transmission name="transmission">
+        <type>transmission_interface/SimpleTransmission</type>
+        <joint name="j2">
+            <hardwareInterface>hardware_interface/EffortJointInterface</hardwareInterface>
+        </joint>
+        <actuator name="motor1">
+            <hardwareInterface>hardware_interface/EffortJointInterface</hardwareInterface>
+            <mechanicalReduction>1</mechanicalReduction>
+        </actuator>
+        </transmission>    <transmission name="transmission">
+        <type>transmission_interface/SimpleTransmission</type>
+        <joint name="j3">
+            <hardwareInterface>hardware_interface/EffortJointInterface</hardwareInterface>
+        </joint>
+        <actuator name="motor1">
+            <hardwareInterface>hardware_interface/EffortJointInterface</hardwareInterface>
+            <mechanicalReduction>1</mechanicalReduction>
+        </actuator>
+    </transmission>
+    <transmission name="transmission">
+        <type>transmission_interface/SimpleTransmission</type>
+        <joint name="j4">
+            <hardwareInterface>hardware_interface/EffortJointInterface</hardwareInterface>
+        </joint>
+        <actuator name="motor1">
+            <hardwareInterface>hardware_interface/EffortJointInterface</hardwareInterface>
+            <mechanicalReduction>1</mechanicalReduction>
+        </actuator>
+    </transmission>
+    <transmission name="transmission">
+        <type>transmission_interface/SimpleTransmission</type>
+        <joint name="j5">
+            <hardwareInterface>hardware_interface/EffortJointInterface</hardwareInterface>
+        </joint>
+        <actuator name="motor1">
+            <hardwareInterface>hardware_interface/EffortJointInterface</hardwareInterface>
+            <mechanicalReduction>1</mechanicalReduction>
+        </actuator>
+        </transmission>    <transmission name="transmission">
+        <type>transmission_interface/SimpleTransmission</type>
+        <joint name="j6">
+            <hardwareInterface>hardware_interface/EffortJointInterface</hardwareInterface>
+        </joint>
+        <actuator name="motor1">
+            <hardwareInterface>hardware_interface/EffortJointInterface</hardwareInterface>
+            <mechanicalReduction>1</mechanicalReduction>
+        </actuator>
+    </transmission>
+    <gazebo>
+        <plugin name="gazebo_ros_control" filename="libgazebo_ros_control.so">
+            <robotNamespace>/my_robotic_arm</robotNamespace>
+        </plugin>
+    </gazebo>
 </robot>

Commit message: Working t123, t456 not working

File: urdf/arm.xacro (robot description, xacro)
@@ -38,7 +38,7 @@
     <xacro:property name="l1" value="0.3"/>
     <xacro:property name="l2" value="1"/>
-    <xacro:property name="l3" value="0.8"/>
-    <xacro:property name="l4" value="0.2"/>
-    <xacro:property name="l5" value="0.2"/>
+    <xacro:property name="l3" value="1"/>
+    <xacro:property name="l4" value="0.00001"/>
+    <xacro:property name="l5" value="0.00001"/>
     <xacro:property name="l6" value="0.2"/>
     <xacro:property name="end_ball_radius" value="0.025"/>
@@ -50,5 +50,5 @@
         <child link="joint1"/>
         <axis xyz="0 0 1"/>
-        <limit velocity="5.0" effort="100" lower="${-pi*0.75}" upper="${pi*0.75}"/>
+        <limit velocity="5.0" effort="100" lower="${-pi*0.95}" upper="${pi*0.95}"/>
         <dynamics damping="0.7"/>
     </joint>
@@ -102,5 +102,5 @@
         <child link="joint2"/>
         <axis xyz="0 0 1 "/>
-        <limit velocity="5.0" effort="100" lower="${-pi*0.75}" upper="${pi*0.75}"/>
+        <limit velocity="5.0" effort="100" lower="${-pi*0.95}" upper="${pi*0.95}"/>
         <dynamics damping="0.7"/>
     </joint>
@@ -154,5 +154,5 @@
         <child link="joint3"/>
         <axis xyz="0 0 1"/>
-        <limit velocity="5.0" effort="100" lower="${-pi*0.75}" upper="${pi*0.75}"/>
+        <limit velocity="5.0" effort="100" lower="${-pi*0.95}" upper="${pi*0.95}"/>
         <dynamics damping="0.7"/>
     </joint>
@@ -206,5 +206,5 @@
         <child link="joint4"/>
         <axis xyz="0 0 1"/>
-        <limit velocity="5.0" effort="100" lower="${-pi*0.75}" upper="${pi*0.75}"/>
+        <limit velocity="5.0" effort="100" lower="${-pi*0.95}" upper="${pi*0.95}"/>
         <dynamics damping="0.7"/>
     </joint>
@@ -258,5 +258,5 @@
         <child link="joint5"/>
         <axis xyz="0 0 1"/>
-        <limit velocity="5.0" effort="100" lower="${-pi*0.75}" upper="${pi*0.75}"/>
+        <limit velocity="5.0" effort="100" lower="${-pi*1.75}" upper="${pi*1.75}"/>
         <dynamics damping="0.7"/>
     </joint>

Commit message: Some changes
Signed-off-by: Yossi Ovcharik <yossiovcharik@gmail.com>

File: urdf/arm.xacro (robot description, xacro)
@@ -34,17 +34,17 @@
     <xacro:property name="M_PI" value="3.141592654"/>
     <xacro:property name="joint_radius" value="0.05"/>
-    <xacro:property name="joint_height" value="0.2"/>
+    <xacro:property name="joint_height" value="0.1"/>
     <xacro:property name="width" value="0.05"/>
     <xacro:property name="l1" value="0.3"/>
-    <xacro:property name="l2" value="1"/>
-    <xacro:property name="l3" value="1"/>
-    <xacro:property name="l4" value="0.00001"/>
-    <xacro:property name="l5" value="0.00001"/>
-    <xacro:property name="l6" value="0.2"/>
+    <xacro:property name="l2" value="0.5"/>
+    <xacro:property name="l3" value="0.5"/>
+    <xacro:property name="l4" value="0.3"/>
+    <xacro:property name="l5" value="0.3"/>
+    <xacro:property name="l6" value="0.3"/>
     <xacro:property name="end_ball_radius" value="0.025"/>
     <!-- Used for fixing robot to Gazebo 'link 1' -->
     <link name="world"/>
     <joint name="j1" type="revolute">
-        <origin xyz="0 0 0.15" rpy="0 0 0"/>
+        <origin xyz="0 0 0.1" rpy="0 0 0"/>
         <parent link="world"/>
         <child link="joint1"/>
@@ -89,5 +89,5 @@
                 <box size="${width} ${width} ${l1}"/>
             </geometry>
-            <material name="darkgreen"/>
+            <material name="black"/>
         </visual>
         <inertial>
@@ -98,5 +98,5 @@
     </link>
     <joint name="j2" type="revolute">
-        <origin xyz="0 0 ${l1}" rpy="${pi*0.0} ${pi*0.5} ${pi*0.0}"/>
+        <origin xyz="0 0 ${l1}" rpy="${0.5*pi} ${-0.0*pi} ${pi*0.0}"/>
         <parent link="joint1"/>
         <child link="joint2"/>
@@ -137,9 +137,9 @@
         </collision>
         <visual>
-            <origin xyz="0 ${l2/2} 0 " rpy="0 0 0"/>
-            <geometry>
-                <box size="${width} ${l2} ${width}"/>
-            </geometry>
-            <material name="darkgreen"/>
+            <origin xyz="${l2/2} 0 0 " rpy="0 0 0"/>
+            <geometry>
+                <box size="${l2} ${width} ${width}"/>
+            </geometry>
+            <material name="black"/>
         </visual>
         <inertial>
@@ -150,5 +150,5 @@
     </link>
     <joint name="j3" type="revolute">
-        <origin xyz="0 ${l2} 0" rpy="${pi*0.0} ${pi*0.0} ${pi*0.5}"/>
+        <origin xyz="${l2} 0 0" rpy="${pi*0.0} ${pi*0.0} ${pi*0.0}"/>
         <parent link="joint2"/>
         <child link="joint3"/>
@@ -193,5 +193,5 @@
                 <box size="${l3} ${width} ${width}"/>
             </geometry>
-            <material name="darkgreen"/>
+            <material name="black"/>
         </visual>
         <inertial>
@@ -245,5 +245,5 @@
                 <box size="${width} ${width} ${l4} "/>
             </geometry>
-            <material name="darkgreen"/>
+            <material name="black"/>
         </visual>
         <inertial>
@@ -258,5 +258,5 @@
         <child link="joint5"/>
         <axis xyz="0 0 1"/>
-        <limit velocity="5.0" effort="100" lower="${-pi*1.75}" upper="${pi*1.75}"/>
+        <limit velocity="5.0" effort="100" lower="${-pi*0.95}" upper="${pi*0.95}"/>
         <dynamics damping="0.7"/>
     </joint>
@@ -297,5 +297,5 @@
                 <box size="${width} ${l5}  ${width}"/>
             </geometry>
-            <material name="green"/>
+            <material name="black"/>
         </visual>
         <inertial>
@@ -341,5 +341,5 @@
             <origin xyz="0 0 0" rpy="0 0 0"/>
             <geometry>
-                <sphere radius="${end_ball_radius}" />
+                <box size="0.1 0.05 0.01"/>
             </geometry>
         </collision>
@@ -347,5 +347,6 @@
             <origin xyz="0 0 0" rpy="0 0 0"/>
             <geometry>
-                <sphere radius="${end_ball_radius}" />
+                <box size="0.1 0.05 0.01"/>
+                <!--<sphere radius="${end_ball_radius}" />-->
             </geometry>
             <material name="blue"/>
